Commit message: Added Gazebo Harmonic ros2_control simulation for Arctos

File: software/arctos_jazzy_ws/src/arctos_description/urdf/arctos_urdf.xacro (robot description, xacro)
@@ -13,5 +13,5 @@
     <origin xyz="0 0 0" rpy="0 0 0"/>
     <geometry>
-      <mesh filename="package://arctos_description/meshes/base_link.stl" scale="0.001 0.001 0.001"/>
+      <mesh filename="file://$(find arctos_description)/meshes/base_link.stl" scale="0.001 0.001 0.001"/>
     </geometry>
     <material name="paint_metallic_blue_2"/>
@@ -20,5 +20,5 @@
     <origin xyz="0 0 0" rpy="0 0 0"/>
     <geometry>
-      <mesh filename="package://arctos_description/meshes/base_link.stl" scale="0.001 0.001 0.001"/>
+      <mesh filename="file://$(find arctos_description)/meshes/base_link.stl" scale="0.001 0.001 0.001"/>
     </geometry>
   </collision>
@@ -33,5 +33,5 @@
     <origin xyz="-0.0 -0.000529 -0.111" rpy="0 0 0"/>
     <geometry>
-      <mesh filename="package://arctos_description/meshes/Link_1_1.stl" scale="0.001 0.001 0.001"/>
+      <mesh filename="file://$(find arctos_description)/meshes/Link_1_1.stl" scale="0.001 0.001 0.001"/>
     </geometry>
     <material name="paint_metallic_blue_2"/>
@@ -40,5 +40,5 @@
     <origin xyz="-0.0 -0.000529 -0.111" rpy="0 0 0"/>
     <geometry>
-      <mesh filename="package://arctos_description/meshes/Link_1_1.stl" scale="0.001 0.001 0.001"/>
+      <mesh filename="file://$(find arctos_description)/meshes/Link_1_1.stl" scale="0.001 0.001 0.001"/>
     </geometry>
   </collision>
@@ -53,5 +53,5 @@
     <origin xyz="0.05713 0.020356 -0.289378" rpy="0 0 0"/>
     <geometry>
-      <mesh filename="package://arctos_description/meshes/Link_2_1.stl" scale="0.001 0.001 0.001"/>
+      <mesh filename="file://$(find arctos_description)/meshes/Link_2_1.stl" scale="0.001 0.001 0.001"/>
     </geometry>
     <material name="paint_metallic_blue_2"/>
@@ -60,5 +60,5 @@
     <origin xyz="0.05713 0.020356 -0.289378" rpy="0 0 0"/>
     <geometry>
-      <mesh filename="package://arctos_description/meshes/Link_2_1.stl" scale="0.001 0.001 0.001"/>
+      <mesh filename="file://$(find arctos_description)/meshes/Link_2_1.stl" scale="0.001 0.001 0.001"/>
     </geometry>
   </collision>
@@ -73,5 +73,5 @@
     <origin xyz="-0.043 0.019045 -0.550385" rpy="0 0 0"/>
     <geometry>
-      <mesh filename="package://arctos_description/meshes/Link_3_1.stl" scale="0.001 0.001 0.001"/>
+      <mesh filename="file://$(find arctos_description)/meshes/Link_3_1.stl" scale="0.001 0.001 0.001"/>
     </geometry>
     <material name="paint_metallic_blue_2"/>
@@ -80,5 +80,5 @@
     <origin xyz="-0.043 0.019045 -0.550385" rpy="0 0 0"/>
     <geometry>
-      <mesh filename="package://arctos_description/meshes/Link_3_1.stl" scale="0.001 0.001 0.001"/>
+      <mesh filename="file://$(find arctos_description)/meshes/Link_3_1.stl" scale="0.001 0.001 0.001"/>
     </geometry>
   </collision>
@@ -93,5 +93,5 @@
     <origin xyz="-1e-06 0.15874 -0.57209" rpy="0 0 0"/>
     <geometry>
-      <mesh filename="package://arctos_description/meshes/Link_4_1.stl" scale="0.001 0.001 0.001"/>
+      <mesh filename="file://$(find arctos_description)/meshes/Link_4_1.stl" scale="0.001 0.001 0.001"/>
     </geometry>
     <material name="paint_metallic_blue_2"/>
@@ -100,5 +100,5 @@
     <origin xyz="-1e-06 0.15874 -0.57209" rpy="0 0 0"/>
     <geometry>
-      <mesh filename="package://arctos_description/meshes/Link_4_1.stl" scale="0.001 0.001 0.001"/>
+      <mesh filename="file://$(find arctos_description)/meshes/Link_4_1.stl" scale="0.001 0.001 0.001"/>
     </geometry>
   </collision>
@@ -113,5 +113,5 @@
     <origin xyz="0.039011 0.279927 -0.570316" rpy="0 0 0"/>
     <geometry>
-      <mesh filename="package://arctos_description/meshes/Link_5_1.stl" scale="0.001 0.001 0.001"/>
+      <mesh filename="file://$(find arctos_description)/meshes/Link_5_1.stl" scale="0.001 0.001 0.001"/>
     </geometry>
     <material name="paint_metallic_blue_2"/>
@@ -120,5 +120,5 @@
     <origin xyz="0.039011 0.279927 -0.570316" rpy="0 0 0"/>
     <geometry>
-      <mesh filename="package://arctos_description/meshes/Link_5_1.stl" scale="0.001 0.001 0.001"/>
+      <mesh filename="file://$(find arctos_description)/meshes/Link_5_1.stl" scale="0.001 0.001 0.001"/>
     </geometry>
   </collision>
@@ -133,5 +133,5 @@
     <origin xyz="-0.000193 0.319847 -0.570316" rpy="0 0 0"/>
     <geometry>
-      <mesh filename="package://arctos_description/meshes/Gripper_1.stl" scale="0.001 0.001 0.001"/>
+      <mesh filename="file://$(find arctos_description)/meshes/Gripper_1.stl" scale="0.001 0.001 0.001"/>
     </geometry>
     <material name="paint_metallic_blue_2"/>
@@ -140,5 +140,5 @@
     <origin xyz="-0.000193 0.319847 -0.570316" rpy="0 0 0"/>
     <geometry>
-      <mesh filename="package://arctos_description/meshes/Gripper_1.stl" scale="0.001 0.001 0.001"/>
+      <mesh filename="file://$(find arctos_description)/meshes/Gripper_1.stl" scale="0.001 0.001 0.001"/>
     </geometry>
   </collision>
@@ -153,5 +153,5 @@
     <origin xyz="-0.000193 0.313762 -0.570316" rpy="0 0 0"/>
     <geometry>
-      <mesh filename="package://arctos_description/meshes/Link_6_1.stl" scale="0.001 0.001 0.001"/>
+      <mesh filename="file://$(find arctos_description)/meshes/Link_6_1.stl" scale="0.001 0.001 0.001"/>
     </geometry>
     <material name="paint_metallic_blue_2"/>
@@ -160,5 +160,5 @@
     <origin xyz="-0.000193 0.313762 -0.570316" rpy="0 0 0"/>
     <geometry>
-      <mesh filename="package://arctos_description/meshes/Link_6_1.stl" scale="0.001 0.001 0.001"/>
+      <mesh filename="file://$(find arctos_description)/meshes/Link_6_1.stl" scale="0.001 0.001 0.001"/>
     </geometry>
   </collision>
@@ -173,5 +173,5 @@
     <origin xyz="-0.007934 0.359845 -0.599867" rpy="0 0 0"/>
     <geometry>
-      <mesh filename="package://arctos_description/meshes/Left_jaw_1.stl" scale="0.001 0.001 0.001"/>
+      <mesh filename="file://$(find arctos_description)/meshes/Left_jaw_1.stl" scale="0.001 0.001 0.001"/>
     </geometry>
     <material name="paint_metallic_blue_2"/>
@@ -180,5 +180,5 @@
     <origin xyz="-0.007934 0.359845 -0.599867" rpy="0 0 0"/>
     <geometry>
-      <mesh filename="package://arctos_description/meshes/Left_jaw_1.stl" scale="0.001 0.001 0.001"/>
+      <mesh filename="file://$(find arctos_description)/meshes/Left_jaw_1.stl" scale="0.001 0.001 0.001"/>
     </geometry>
   </collision>
@@ -193,5 +193,5 @@
     <origin xyz="-0.007934 0.359845 -0.539867" rpy="0 0 0"/>
     <geometry>
-      <mesh filename="package://arctos_description/meshes/Right_jaw_1.stl" scale="0.001 0.001 0.001"/>
+      <mesh filename="file://$(find arctos_description)/meshes/Right_jaw_1.stl" scale="0.001 0.001 0.001"/>
     </geometry>
     <material name="paint_metallic_blue_2"/>
@@ -200,5 +200,5 @@
     <origin xyz="-0.007934 0.359845 -0.539867" rpy="0 0 0"/>
     <geometry>
-      <mesh filename="package://arctos_description/meshes/Right_jaw_1.stl" scale="0.001 0.001 0.001"/>
+      <mesh filename="file://$(find arctos_description)/meshes/Right_jaw_1.stl" scale="0.001 0.001 0.001"/>
     </geometry>
   </collision>
@@ -259,3 +259,45 @@
   <limit upper="0.015" lower="0.0" effort="100" velocity="100"/>
 </joint>
+<ros2_control name="ArctosSystem" type="system">
+  <hardware>
+    <plugin>gz_ros2_control/GazeboSimSystem</plugin>
+  </hardware>
+  <joint name="joint1">
+    <command_interface name="position"/>
+    <state_interface name="position"/>
+    <state_interface name="velocity"/>
+  </joint>
+  <joint name="joint2">
+    <command_interface name="position"/>
+    <state_interface name="position"/>
+    <state_interface name="velocity"/>
+  </joint>
+  <joint name="joint3">
+    <command_interface name="position"/>
+    <state_interface name="position"/>
+    <state_interface name="velocity"/>
+  </joint>
+  <joint name="joint4">
+    <command_interface name="position"/>
+    <state_interface name="position"/>
+    <state_interface name="velocity"/>
+  </joint>
+  <joint name="joint5">
+    <command_interface name="position"/>
+    <state_interface name="position"/>
+    <state_interface name="velocity"/>
+  </joint>
+  <joint name="joint6">
+    <command_interface name="position"/>
+    <state_interface name="position"/>
+    <state_interface name="velocity"/>
+  </joint>
+</ros2_control>
+<gazebo>
+  <plugin
+    filename="libgz_ros2_control-system.so"
+    name="gz_ros2_control::GazeboSimROS2ControlPlugin">
+    <parameters>$(find arctos_description)/config/arctos_controllers.yaml</parameters>
+  </plugin>
+</gazebo>
 </robot>

Commit message: Stabilized Gazebo simulation launch and joint limits

File: software/arctos_jazzy_ws/src/arctos_description/urdf/arctos_urdf.xacro (robot description, xacro)
@@ -204,9 +204,10 @@
   </collision>
 </link>
-<joint name="joint1" type="continuous">
+<joint name="joint1" type="revolute">
   <origin xyz="0.0 0.000529 0.111" rpy="0 0 0"/>
   <parent link="base_link"/>
   <child link="Link_1_1"/>
   <axis xyz="-0.0 0.0 1.0"/>
+  <limit lower="-3.14" upper="3.14" effort="100" velocity="1.5"/>
 </joint>
 <joint name="joint2" type="continuous">
@@ -215,4 +216,5 @@
   <child link="Link_2_1"/>
   <axis xyz="1.0 -0.0 -0.0"/>
+  <limit lower="-1.57" upper="1.57" effort="100" velocity="1.5"/>
 </joint>
 <joint name="joint3" type="continuous">
@@ -221,4 +223,5 @@
   <child link="Link_3_1"/>
   <axis xyz="-1.0 -0.0 0.0"/>
+  <limit lower="-2.0" upper="2.0" effort="100" velocity="1.5"/>
 </joint>
 <joint name="joint4" type="continuous">
@@ -227,4 +230,5 @@
   <child link="Link_4_1"/>
   <axis xyz="-0.0 1.0 -0.0"/>
+  <limit lower="-3.14" upper="3.14" effort="80" velocity="2.0"/>
 </joint>
 <joint name="joint5" type="continuous">
@@ -233,4 +237,5 @@
   <child link="Link_5_1"/>
   <axis xyz="-1.0 -0.0 0.0"/>
+  <limit lower="-2.0" upper="2.0" effort="80" velocity="2.0"/>
 </joint>
 <joint name="gripper" type="fixed">
@@ -244,4 +249,5 @@
   <child link="Link_6_1"/>
   <axis xyz="-0.0 1.0 -0.0"/>
+  <limit lower="-3.14" upper="3.14" effort="50" velocity="2.5"/>
 </joint>
 <joint name="jaw1" type="prismatic">

Commit message: Anchor Arctos base to world in Gazebo

File: software/arctos_jazzy_ws/src/arctos_description/urdf/arctos_urdf.xacro (robot description, xacro)
@@ -4,4 +4,11 @@
 <xacro:include filename="$(find arctos_description)/urdf/arctos_urdf.trans" />
 <xacro:include filename="$(find arctos_description)/urdf/arctos_urdf.gazebo" />
+<!-- Anchor robot base to the Gazebo world frame -->
+<link name="world"/>
+<joint name="world_to_base" type="fixed">
+  <parent link="world"/>
+  <child link="base_link"/>
+  <origin xyz="0 0 0" rpy="0 0 0"/>
+</joint>
 <link name="base_link">
   <inertial>
